File: 1P/1 Player.kicad_pcb (KiCad board)
At the start: 2 copper layers, 18.8 x 32.8 mm, 3 parts

Commit message: 12341234
qwr1234`12ef
Routing:
- net /DATA1: track 12.3 -> 16.1 mm, vias 0 -> 1
- added copper zone on F.Cu, net /GND
